Commit message: packages update

File: erc_ros2_navigation/urdf/erc_bot.urdf (robot description, URDF)
Before this commit: robot mogi_bot, 8 links, 7 joints
Links:
- removed link imu_link
- removed link left_wheel
- removed link right_wheel
- added link front_left_wheel, mass 5.0; collision cylinder length=.05 radius=.1; visual mesh filename=package://erc_ros2_navigation/meshes/IronManWheelLeftFront.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
- added link front_right_wheel, mass 5.0; collision cylinder length=.05 radius=.1; visual mesh filename=package://erc_ros2_navigation/meshes/IronManWheelRightFront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
- added link rear_left_wheel, mass 5.0; collision cylinder length=.05 radius=.1; visual mesh filename=package://erc_ros2_navigation/meshes/IronManWheelRightFront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
- added link rear_right_wheel, mass 5.0; collision cylinder length=.05 radius=.1; visual mesh filename=package://erc_ros2_navigation/meshes/IronManWheelLeftFront.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
- link base_link: geometry collision box size=.4 .2 .1; visual mesh filename=package://erc_ros2_navigation/meshes/IronMan_ROS_Body.dae
- link scan_link: geometry collision box size=.1 .1 .1; visual mesh filename=package://erc_ros2_navigation/meshes/lidar.dae
Joints:
- removed joint imu_joint
- removed joint left_wheel_joint
- removed joint right_wheel_joint
- added joint front_left_wheel_joint: type continuous, parent base_link, child front_left_wheel, origin xyz=0.15 0.15 0 rpy=0 0 0, axis 0 1 0, limit effort=100 velocity=10
- added joint front_right_wheel_joint: type continuous, parent base_link, child front_right_wheel, origin xyz=0.15 -0.15 0 rpy=0 0 0, axis 0 1 0, limit effort=100 velocity=10
- added joint rear_left_wheel_joint: type continuous, parent base_link, child rear_left_wheel, origin xyz=-0.15 0.15 0 rpy=0 0 0, axis 0 1 0, limit effort=100 velocity=10
- added joint rear_right_wheel_joint: type continuous, parent base_link, child rear_right_wheel, origin xyz=-0.15 -0.15 0 rpy=0 0 0, axis 0 1 0, limit effort=100 velocity=10
